File: herblove.kicad_pcb (KiCad board)
At the start: 2 copper layers, 3.2 x 3.2 mm, 6 parts, among them J1 Micro_SD_Card, SW1 SW_Push, SW2 SW_SPDT, U1 bme280, U2 C3 Pico, U3 hw357

Commit message: Add final components
Parts:
- added BT1: Battery_Cell, Connector_JST:JST_PH_B2B-PH-K_1x02_P2.00mm_Vertical, F.Cu at (137.1, 43.9)
- added J2: 12V Valve, Connector_PinHeader_2.54mm:PinHeader_1x02_P2.54mm_Vertical, F.Cu at (144.3, 43.5)
- added J3: Empty Sensor, Connector_PinHeader_2.54mm:PinHeader_1x02_P2.54mm_Vertical, F.Cu at (149.0, 43.5)
- added J4: Switched Battery, Connector_JST:JST_PH_B2B-PH-K_1x02_P2.00mm_Vertical, F.Cu at (137.1, 50.4)
- added J5: Solar Panel, Connector_JST:JST_PH_B2B-PH-K_1x02_P2.00mm_Vertical, F.Cu at (119.0, 36.0)
- added J6: Micro_SD_Card, sd-card:sd-card, F.Cu at (53.0, 51.0)
- added SW3: SW_Push, pts636:pts636, F.Cu at (102.6, 38.0)
- moved U1 55.4 mm to (122.7, 104.2)
- moved U3 50.8 mm to (92.4, 93.7), turned to 180 degrees
- moved J1 45.8 mm to (81.0, 110.0), turned to 180 degrees
- moved U2 26.9 mm to (103.0, 107.0)
Connections:
- J1 pad 9: unconnected-(J1-SHIELD-Pad9) -> GND
- SW1 pad 1: unconnected-(SW1-Pad1) -> SWITCH_A
- SW1 pad 2: unconnected-(SW1-Pad2) -> GND
- SW2 pad 1: unconnected-(SW2-A-Pad1) -> Net-(BT1-+)
- SW2 pad 2: unconnected-(SW2-B-Pad2) -> Net-(J4-Pin_2)
- U1 pad 1: unconnected-(U1-VIN-Pad1) -> +3V3
- U1 pad 3: unconnected-(U1-SCL-Pad3) -> SCL
- U1 pad 4: unconnected-(U1-SDA-Pad4) -> SDA
- U2 pad 2: unconnected-(U2-GND-Pad2) -> GND
- U2 pad 5: unconnected-(U2-SDA/IO8-Pad5) -> SDA
- U2 pad 6: unconnected-(U2-SCL/IO10-Pad6) -> SCL
- U2 pad 9: unconnected-(U2-3V3-Pad9) -> +3V3
- U3 pad 1: unconnected-(U3-IN+-Pad1) -> Net-(J5-Pin_2)
- U3 pad 2: unconnected-(U3-IN--Pad2) -> GND
- U3 pad 3: unconnected-(U3-O+-Pad3) -> SWITCHED_12V
- U3 pad 5: unconnected-(U3-B+-Pad5) -> Net-(BT1-+)
- U3 pad 6: unconnected-(U3-B--Pad6) -> Net-(BT1--)
Other:
- board size 3.2 x 3.2 mm -> 90 x 54 mm

Commit message: Finalise routing
Parts:
- added J7: Conn_01x04_Pin, Connector_PinHeader_2.54mm:PinHeader_1x04_P2.54mm_Vertical, B.Cu at (111.0, 110.5)
- added R1: 1k, Resistor_THT:R_Axial_DIN0207_L6.3mm_D2.5mm_P7.62mm_Horizontal, F.Cu at (109.0, 86.2)
- added R2: 1k, Resistor_THT:R_Axial_DIN0207_L6.3mm_D2.5mm_P7.62mm_Horizontal, F.Cu at (113.8, 78.5)
- added R3: 1k, Resistor_THT:R_Axial_DIN0207_L6.3mm_D2.5mm_P7.62mm_Horizontal, F.Cu at (118.2, 86.2)
- added R4: 1k, Resistor_THT:R_Axial_DIN0207_L6.3mm_D2.5mm_P7.62mm_Horizontal, F.Cu at (106.2, 92.0)
- J1: value Micro_SD_Card -> Conn_01x01_Pin; footprint sd-card:sd-card -> Connector_PinHeader_2.54mm:PinHeader_1x01_P2.54mm_Vertical
- moved BT1 76.6 mm to (71.2, 83.0), turned to -90 degrees
- moved J4 74.8 mm to (78.2, 96.6), turned to 180 degrees
- moved J6 67.1 mm to (86.8, 109.0), turned to 180 degrees
- moved J5 62.3 mm to (71.2, 76.0), turned to -90 degrees
- moved SW2 61.0 mm to (70.0, 90.5)
- moved SW3 60.2 mm to (122.0, 95.0), turned to 90 degrees
- moved J3 42.5 mm to (120.5, 75.0), turned to 180 degrees
- moved J2 42.3 mm to (112.5, 71.2), turned to -90 degrees
- moved SW1 22.5 mm to (122.0, 78.8), turned to -90 degrees
- moved J1 15.3 mm to (89.0, 97.0), turned to 0 degrees
- moved U3 14.1 mm to (106.5, 93.1)
- moved U1 4.54 mm to (118.2, 104.0)
- moved U2 0.71 mm to (103.5, 106.5)
Connections:
- J1 pad 1: unconnected-(J1-DAT2-Pad1) -> ENABLE_12V
- U1 pad 2: unconnected-(U1-GND-Pad2) -> GND
- U2 pad 10: unconnected-(U2-IO5-Pad10) -> SPI_CS
- U2 pad 11: unconnected-(U2-IO4/MOSI-Pad11) -> SPI_MOSI
- U2 pad 12: unconnected-(U2-IO0/ADC/MISO-Pad12) -> SPI_CLK
- U2 pad 13: unconnected-(U2-IO1/ADC/SCK-Pad13) -> SPI_MISO
- U2 pad 14: unconnected-(U2-IO2-Pad14) -> ENABLE_12V
- U2 pad 3: unconnected-(U2-IO6-Pad3) -> BUTTONS_ADC
Routing:
- net GND: track 0.00 -> 134.5 mm
- net +3V3: track 0.00 -> 119.0 mm
- net BUTTONS_ADC: track 0.00 -> 40.8 mm
- net Net-(BT1-+): track 0.00 -> 30.3 mm
- net Net-(J5-Pin_2): track 0.00 -> 22.9 mm
- net EMPTY_SENSOR: track 0.00 -> 15.7 mm
- net SWITCH_B: track 0.00 -> 15.2 mm
- net Net-(BT1--): track 0.00 -> 10.3 mm
- net ENABLE_12V: track 0.00 -> 10.0 mm
- net SDA: track 0.00 -> 8.14 mm
- net SCL: track 0.00 -> 8.14 mm
- net Net-(J4-Pin_2): track 0.00 -> 7.62 mm
- net SPI_MISO: track 0.00 -> 6.47 mm
- net SPI_CLK: track 0.00 -> 5.86 mm
- net SPI_CS: track 0.00 -> 5.48 mm
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- added copper zone on B.Cu, net GND
Other:
- board size 90 x 54 mm -> 56 x 51 mm
